File: hardware/countdown_debug.brd (EAGLE design)
At the start: 38 x 40 mm, 30 parts, among them J1 BURNIN, J2 USB, J3 LiPo, J4 OLED, J5 TOP, J6 BASE, U1 DS3231MZ+TRL_SOIC8, U2 ATMEGA328P-AUR, U3 MCP73831T, U4 BL1551

Commit message: make debug version
Parts:
- added J7: (no value), scono:1X04
- J5: value TOP -> (none); device scono:1X03_NO_SILK -> scono:1X02
- J6: value BASE -> (none); device scono:1X03_NO_SILK -> scono:1X04
- moved R7 27.7 mm to (-6.25, -30.2), turned to 0 degrees
- moved D2 22.6 mm to (-2.25, -31.2), turned to 0 degrees
- moved J6 9.17 mm to (9.25, 0.25), turned to 180 degrees
- moved J5 1.80 mm to (19.8, 5.50)
- moved D1 1.00 mm to (15.5, -18.0)
- moved U3 0.75 mm to (13.0, -18.0)
- moved R1 0.56 mm to (15.0, -20.8), turned to 0 degrees
- moved C4 0.50 mm to (15.0, -15.2)
- moved R2 0.50 mm to (12.5, -15.2)
- moved C3 0.25 mm to (12.5, -20.8)
- moved J2 0.25 mm to (20.8, -21.2)
- moved BT1 0.10 mm to (5.75, -11.5)
Connections:
- removed net GND_BOT: BT1.3, C3.1, C4.1, J2.5, J3.1, J6.1, R2.1, R7.1, U3.2
- removed net GND_TOP: C1.1, C2.1, C5.1, C6.1, C7.1, J1.GND, J4.1, J5.1, R4.2, R5.2, R6.1, U1.5, U2.21, U2.3, U2.5, U4.2
- removed net VCC_BOT: J6.3, U$1.1
- removed net VCC_TOP: C5.2, C6.2, J1.3.3V, J4.2, J5.3, R3.1, SW_INT.P$1, U2.4, U2.6, U4.1, U4.4
- removed net V_BAT_BOT: BT1.1, BT1.2, J6.2
- removed net V_BAT_TOP: J5.2, U1.6
- new net GND: BT1.3, C1.1, C2.1, C3.1, C4.1, C5.1, C6.1, C7.1, J1.GND, J2.5, J3.1, J4.1, R2.1, R4.2, R5.2, R6.1, R7.1, U1.5, U2.21, U2.3, U2.5, U3.2, U4.2
- new net VCC: C5.2, C6.2, J1.3.3V, J4.2, R3.1, SW_INT.P$1, U$1.1, U2.4, U2.6, U4.1, U4.4
- new net V_BAT: BT1.1, BT1.2, U1.6
- net EN_CLK: now also J6.1
- net INT_WAKE: now also J6.4
- net MISO: now also J7.3
- net MOSI: now also J7.4
- net RST: now also J7.1
- net SCK: now also J7.2
- net SCL: now also J6.3
- net SDA: now also J6.2
- net XTAL1: now also J5.2
- net XTAL2: now also J5.1
Routing:
- net VCC: track 0.00 -> 96.0 mm, vias 0 -> 7
- net VCC_TOP: track 71.9 -> 0.00 mm, vias 7 -> 0
- net V_BAT: track 0.00 -> 51.9 mm, vias 0 -> 4
- net V_BAT_BOT: track 36.3 -> 0.00 mm, vias 2 -> 0
- net EN_CLK: track 27.1 -> 52.6 mm, vias 4 -> 7
- net RST: track 18.5 -> 43.1 mm, vias 2 -> 5
- net VCC_BOT: track 23.8 -> 0.00 mm
- net V_BAT_TOP: track 14.2 -> 0.00 mm, vias 1 -> 0
- net SCL: track 31.2 -> 43.6 mm, vias 4 -> 5
- net SDA: track 41.0 -> 53.2 mm, vias 4 -> 5
- net GND: track 0.00 -> 12.0 mm, vias 0 -> 5
- net INT_WAKE: track 8.00 -> 17.5 mm
- net SCK: track 18.3 -> 26.7 mm
- net GND_TOP: track 7.64 -> 0.00 mm, vias 3 -> 0
- net MISO: track 19.0 -> 25.7 mm
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- added copper zone on layer 1, net GND
- added copper zone on layer 16, net GND
- removed copper zone on layer 1, net GND_BOT
- removed copper zone on layer 16, net GND_BOT
- removed copper zone on layer 1, net GND_TOP
- removed copper zone on layer 16, net GND_TOP
Other:
- outline, holes or cut-outs redrawn
- board text added: "I2C"
- board text added: "ICP"
- board text added: "INT"
- board text added: "SWITCH"
- board text added: "XTAL"

Commit message: prepare for order
Parts:
- removed BT1: BK-916-TR, scono:BAT_BK-916-TR
- removed C3, C4: 4.7uF, scono:0402-CAP
- removed D1, D2: (no value), scono:LED-0603
- removed J2: USB, scono:FCI_10103594-0001LF
- removed R1, R7: 330R, scono:R0402
- removed R2: 125k, scono:R0402
- removed U3: MCP73831T, scono:SOT-23-5
- added BT2: BK-916-TR, scono:BAT_BK-916-TR
- added C10, C11: 4.7uF, scono:0402-CAP
- added D3, D4: (no value), scono:LED-0603
- added J9: USB, scono:FCI_10103594-0001LF
- added R14, R8: 330R, scono:R0402
- added R9: 51k, scono:R0402
- added U6: MCP73831T, scono:SOT-23-5
- renumbered J3 to J10, U$1 to U$2
Connections:
- removed net N$2: D2.C, R7.2
- removed net N$4: D1.C, R1.2
- removed net PROG: R2.2, U3.5
- new net N$3: D3.C, R8.2
- new net N$6: D4.C, R14.2
- new net PROG1: R9.2, U6.5
- net GND: now also BT2.3, C10.1, C11.1, J9.5, R14.1, R9.1, U6.2; no longer BT1.3, C3.1, C4.1, J2.5, R2.1, R7.1, U3.2
- net STAT: now also D4.A, R8.1, U6.1; no longer D2.A, R1.1, U3.1
- net VBAT_CHARGE: now also C10.2, U6.3; no longer C3.2, U3.3
- net VUSB: now also C11.2, D3.A, J9.1, U6.4; no longer C4.2, D1.A, J2.1, U3.4
- net V_BAT: now also BT2.1, BT2.2; no longer BT1.1, BT1.2
Routing:
- net STAT: track 6.13 -> 9.64 mm, vias 2 -> 0
- net N$6: track 0.00 -> 2.02 mm
- net N$4: track 1.94 -> 0.00 mm
- net VBAT_CHARGE: track 24.1 -> 22.4 mm, vias 2 -> 1
- net PROG: track 1.53 -> 0.00 mm
- net PROG1: track 0.00 -> 1.47 mm
- net N$3: track 0.00 -> 1.41 mm

Commit message: jlc order done
Parts:
- added C3: 0.1uF, scono:0402-CAP
- moved BT2 23.0 mm to (5.65, 11.5)
- moved C1 23.0 mm to (18.5, 33.0)
- moved C10 23.0 mm to (12.2, 2.25)
- moved C11 23.0 mm to (14.5, 7.75)
- moved C2 23.0 mm to (26.0, 33.0)
- moved C5 23.0 mm to (17.0, 33.5)
- moved C6 23.0 mm to (5.00, 33.0)
- moved C7 23.0 mm to (30.5, 35.2)
- moved D3 23.0 mm to (14.5, 5.00)
- moved D4 23.0 mm to (16.0, 5.00)
- moved J1 23.0 mm to (18.8, 36.0)
- moved J10 23.0 mm to (13.5, 16.0)
- moved J4 23.0 mm to (35.5, 30.0)
- moved J5 23.0 mm to (19.8, 28.5)
- moved J6 23.0 mm to (9.25, 23.2)
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Connections:
- net GND: now also C3.1
- net INT_WAKE: now also C3.2
Other:
- outline, holes or cut-outs redrawn
