File: hardware/countdown_debug.sch (EAGLE design)
At the start: 30 parts, among them J1 BURNIN, J2 USB, J3 LiPo, J4 OLED, J5 TOP, J6 BASE, U1 DS3231MZ+TRL_SOIC8, U2 ATMEGA328P-AUR, U3 MCP73831T, U4 BL1551

Commit message: make debug version
Parts:
- added J7: (no value), scono:CONN_04
- J5: value TOP -> (none); device scono:CONN_031X03_NO_SILK -> scono:CONN_02
- J6: value BASE -> (none); device scono:CONN_031X03_NO_SILK -> scono:CONN_04
Connections:
- removed net GND_BOT: BT1.-, C3.1, C4.1, J2.UGND, J3.1, J6.1, R2.1, R7.1, U3.GND
- removed net GND_TOP: C1.1, C2.1, C5.1, C6.1, C7.1, J1.GND, J4.1, J5.1, R4.2, R5.2, R6.1, U1.GND, U2.GND, U4.GND
- removed net VCC_BOT: J6.3, U$1.A
- removed net VCC_TOP: C5.2, C6.2, J1.VCC, J4.2, J5.3, R3.1, SW_INT.P, U2.VCC, U4.A1, U4.B
- removed net V_BAT_BOT: BT1.+, J6.2
- removed net V_BAT_TOP: J5.2, U1.VBAT
- new net GND: BT1.-, C1.1, C2.1, C3.1, C4.1, C5.1, C6.1, C7.1, J1.GND, J2.UGND, J3.1, J4.1, R2.1, R4.2, R5.2, R6.1, R7.1, U1.GND, U2.GND, U3.GND, U4.GND
- new net VCC: C5.2, C6.2, J1.VCC, J4.2, R3.1, SW_INT.P, U$1.A, U2.VCC, U4.A1, U4.B
- new net V_BAT: BT1.+, U1.VBAT
- net EN_CLK: now also J6.1
- net INT_WAKE: now also J6.4
- net MISO: now also J7.3
- net MOSI: now also J7.4
- net RST: now also J7.1
- net SCK: now also J7.2
- net SCL: now also J6.3
- net SDA: now also J6.2
- net XTAL1: now also J5.2
- net XTAL2: now also J5.1

Commit message: prepare for order
Parts:
- removed BT1: BK-916-TR, scono:BK-916-TR
- removed C3, C4: 4.7uF, scono:CAP0402-CAP
- removed D1, D2: (no value), scono:LED0603
- removed J2: USB, scono:USB
- removed J3: LiPo, scono:CONN_02
- removed R1, R7: 330R, scono:R-US_R0402
- removed R2: 125k, scono:R-US_R0402
- removed U$1: CL-SB-12C-12, scono:CL-SB-12C-12
- removed U3: MCP73831T, scono:MCP73831T
- added BT2: BK-916-TR, scono:BK-916-TR
- added C10, C11: 4.7uF, scono:CAP0402-CAP
- added D3, D4: (no value), scono:LED0603
- added J10: LiPo, scono:CONN_02
- added J9: USB, scono:USB
- added R14, R8: 330R, scono:R-US_R0402
- added R9: 51k, scono:R-US_R0402
- added U$2: CL-SB-12C-12, scono:CL-SB-12C-12
- added U6: MCP73831T, scono:MCP73831T
Connections:
- removed net N$2: D2.C, R7.2
- removed net N$4: D1.C, R1.2
- removed net PROG: R2.2, U3.PROG
- new net N$3: D3.C, R8.2
- new net N$6: D4.C, R14.2
- new net PROG1: R9.2, U6.PROG
- net BAT+: now also J10.2, U$2.OUT; no longer J3.2, U$1.OUT
- net GND: now also BT2.-, C10.1, C11.1, J10.1, J9.UGND, R14.1, R9.1, U6.GND; no longer BT1.-, C3.1, C4.1, J2.UGND, J3.1, R2.1, R7.1, U3.GND
- net STAT: now also D4.A, R8.1, U6.STAT; no longer D2.A, R1.1, U3.STAT
- net VBAT_CHARGE: now also C10.2, U$2.B, U6.VBAT; no longer C3.2, U$1.B, U3.VBAT
- net VCC: now also U$2.A; no longer U$1.A
- net VUSB: now also C11.2, D3.A, J9.VUSB, U6.VDD; no longer C4.2, D1.A, J2.VUSB, U3.VDD
- net V_BAT: now also BT2.+; no longer BT1.+

Commit message: jlc order done
Parts:
- added C3: 0.1uF, scono:CAP0402-CAP
Connections:
- net GND: now also C3.1
- net INT_WAKE: now also C3.2
Changed lines of the file:
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@@
 <part name="SUPPLY2" library="scono" library_urn="urn:adsk.eagle:library:14850048" deviceset="GND" device=""/>
 <part name="SUPPLY3" library="scono" library_urn="urn:adsk.eagle:library:14850048" deviceset="GND" device=""/>
+<part name="C3" library="scono" library_urn="urn:adsk.eagle:library:14850048" deviceset="CAP" device="0402-CAP" package3d_urn="urn:adsk.eagle:package:14850678/3" value="0.1uF"/>
 </parts>
 <sheets>
@@
 <instance part="SUPPLY2" gate="GND" x="162.56" y="55.88" smashed="yes"/>
 <instance part="SUPPLY3" gate="GND" x="68.58" y="33.02" smashed="yes"/>
+<instance part="C3" gate="G$1" x="228.6" y="116.84" smashed="yes" rot="R90">
+<attribute name="NAME" x="227.076" y="115.57" size="1.016" layer="95" rot="R90"/>
+<attribute name="VALUE" x="231.14" y="115.57" size="1.016" layer="96" rot="R90"/>
+</instance>
 </instances>
 <busses>
@@
 <label x="220.98" y="109.22" size="1.778" layer="95"/>
 <pinref part="SUPPLY6" gate="GND" pin="GND"/>
+<pinref part="C3" gate="G$1" pin="1"/>
+<wire x1="228.6" y1="114.3" x2="228.6" y2="111.76" width="0.1524" layer="91"/>
+<wire x1="228.6" y1="111.76" x2="220.98" y2="111.76" width="0.1524" layer="91"/>
+<junction x="220.98" y="111.76"/>
 </segment>
 <segment>
@@
 <pinref part="R6" gate="G$1" pin="2"/>
 <label x="220.98" y="121.92" size="1.778" layer="95"/>
-</segment>
-<segment>
+<pinref part="C3" gate="G$1" pin="2"/>
+<wire x1="220.98" y1="119.38" x2="228.6" y2="119.38" width="0.1524" layer="91"/>
+<junction x="220.98" y="119.38"/>
+</segment>
+<segment>
